File: KiCad Work/PracticumEQLightBar/PracticumEQLightBar.kicad_pcb (KiCad board)
At the start: 2 copper layers, 300 x 114.6 mm, 52 parts, among them U1 TEENSY 4.1, U2 TEENSY AUDIO ADAPTER BOARD RE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, U4 SN74AHCT125N

Commit message: Commited wrong version last time
Parts:
- added REF**: MountingHole_2.2mm_M2_ISO7380_Pad, MountingHole:MountingHole_2.2mm_M2_ISO7380_Pad, F.Cu at (30.5, 138.4)
- added REF**: MountingHole_2.2mm_M2_ISO7380_Pad, MountingHole:MountingHole_2.2mm_M2_ISO7380_Pad, F.Cu at (323.9, 138.4)
- added REF**: MountingHole_2.2mm_M2_ISO7380_Pad, MountingHole:MountingHole_2.2mm_M2_ISO7380_Pad, F.Cu at (323.9, 73.7)
- added REF**: MountingHole_2.2mm_M2_ISO7380_Pad, MountingHole:MountingHole_2.2mm_M2_ISO7380_Pad, F.Cu at (30.5, 73.7)
- added REF**: MountingHole_2.2mm_M2_ISO7380_Pad, MountingHole:MountingHole_2.2mm_M2_ISO7380_Pad, F.Cu at (177.8, 108.0)
- added TP1: TestPoint_Alt, TestPoint:TestPoint_Pad_1.5x1.5mm, F.Cu at (43.2, 109.2)
- added TP2: TestPoint_Alt, TestPoint:TestPoint_Pad_1.5x1.5mm, F.Cu at (47.0, 113.0)
- U1: footprint EQLightBarLibrary:MODULE_DEV-16771 -> EQLightBarLibrary:Double PinSocket_1x24_P2.54mm_Vertical (Teensy 4_1)
- moved U2 48.8 mm to (67.3, 35.6), turned to 0 degrees
- moved U1 18.9 mm to (50.8, 91.4), turned to 90 degrees
- moved U4 11.1 mm to (43.2, 129.5), turned to 180 degrees
- moved D11 0.42 mm to (150.3, 132.4)
- moved D13 0.42 mm to (168.1, 132.4)
- moved D15 0.42 mm to (185.8, 132.4)
- moved D17 0.42 mm to (203.6, 132.4)
- moved D19 0.42 mm to (221.4, 132.4)
- moved D21 0.42 mm to (239.2, 132.4)
- moved D25 0.42 mm to (274.8, 132.4)
- moved D26 0.42 mm to (283.6, 132.4)
- moved D27 0.42 mm to (292.5, 132.4)
- moved D29 0.42 mm to (310.3, 132.4)
- moved D30 0.42 mm to (296.3, 123.5)
- moved D31 0.42 mm to (287.4, 123.5)
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Connections:
- D1 pad 1: /5.0V DATA -> Net-(D1-DI)
- D1 pad 2: unconnected-(D1-CI-Pad2) -> Net-(D1-CI)
- D1 pad 4: Net-(D1-VCC) -> 5V USB
- D10 pad 4: Net-(D1-VCC) -> 5V USB
- D11 pad 4: Net-(D1-VCC) -> 5V USB
- D12 pad 4: Net-(D1-VCC) -> 5V USB
- D13 pad 4: Net-(D1-VCC) -> 5V USB
- D14 pad 4: Net-(D1-VCC) -> 5V USB
- D15 pad 4: Net-(D1-VCC) -> 5V USB
- D16 pad 4: Net-(D1-VCC) -> 5V USB
- D17 pad 4: Net-(D1-VCC) -> 5V USB
- D18 pad 4: Net-(D1-VCC) -> 5V USB
- D19 pad 4: Net-(D1-VCC) -> 5V USB
- D2 pad 4: Net-(D1-VCC) -> 5V USB
- D20 pad 4: Net-(D1-VCC) -> 5V USB
- D21 pad 4: Net-(D1-VCC) -> 5V USB
- D22 pad 4: Net-(D1-VCC) -> 5V USB
- D23 pad 4: Net-(D1-VCC) -> 5V USB
- D24 pad 4: Net-(D1-VCC) -> 5V USB
- D25 pad 4: Net-(D1-VCC) -> 5V USB
- D26 pad 4: Net-(D1-VCC) -> 5V USB
- D27 pad 4: Net-(D1-VCC) -> 5V USB
- D28 pad 4: Net-(D1-VCC) -> 5V USB
- D29 pad 4: Net-(D1-VCC) -> 5V USB
- D3 pad 4: Net-(D1-VCC) -> 5V USB
- D30 pad 4: Net-(D1-VCC) -> 5V USB
- D31 pad 4: Net-(D1-VCC) -> 5V USB
- D32 pad 4: Net-(D1-VCC) -> 5V USB
- D33 pad 4: Net-(D1-VCC) -> 5V USB
- D34 pad 4: Net-(D1-VCC) -> 5V USB
- D35 pad 4: Net-(D1-VCC) -> 5V USB
- D36 pad 4: Net-(D1-VCC) -> 5V USB
- D37 pad 4: Net-(D1-VCC) -> 5V USB
- D38 pad 4: Net-(D1-VCC) -> 5V USB
- D39 pad 4: Net-(D1-VCC) -> 5V USB
- D4 pad 4: Net-(D1-VCC) -> 5V USB
- D40 pad 4: Net-(D1-VCC) -> 5V USB
- D41 pad 4: Net-(D1-VCC) -> 5V USB
- D42 pad 4: Net-(D1-VCC) -> 5V USB
- D43 pad 4: Net-(D1-VCC) -> 5V USB
- D44 pad 4: Net-(D1-VCC) -> 5V USB
- D45 pad 4: Net-(D1-VCC) -> 5V USB
- D46 pad 4: Net-(D1-VCC) -> 5V USB
- D47 pad 4: Net-(D1-VCC) -> 5V USB
- D48 pad 4: Net-(D1-VCC) -> 5V USB
- D49 pad 4: Net-(D1-VCC) -> 5V USB
- D5 pad 4: Net-(D1-VCC) -> 5V USB
- D6 pad 4: Net-(D1-VCC) -> 5V USB
- D7 pad 4: Net-(D1-VCC) -> 5V USB
- D8 pad 4: Net-(D1-VCC) -> 5V USB
- D9 pad 4: Net-(D1-VCC) -> 5V USB
- U1 pad 24: unconnected-(U1-A10-Pad24) -> /CLOCK
- U4 pad 2: /3.3V DATA -> /CLOCK
- U4 pad 3: /5.0V DATA -> Net-(D1-CI)
- U4 pad 4: unconnected-(U4-2~{OE}-Pad4) -> GND
- U4 pad 5: unconnected-(U4-2A-Pad5) -> /3.3V DATA
- U4 pad 6: unconnected-(U4-2Y-Pad6) -> Net-(D1-DI)
Routing:
- net 5V USB: track 93.8 -> 0.00 mm
- net /CLOCK: track 0.00 -> 78.0 mm
- net /5.0V DATA: track 39.1 -> 0.00 mm
- net /3.3V DATA: track 43.0 -> 66.5 mm
- net Net-(D1-DI): track 0.00 -> 14.6 mm
- net Net-(D1-CI): track 0.00 -> 12.0 mm
Other:
- board size 300 x 114.6 mm -> 300 x 71.4 mm
- board text added: "The GND/5V edge of the board should probably line up with the left side of the PCB so that both the built-in aux jack and micro-usb port can be flush with the enclosure"
- board text added: "WE REALLY REALLY NEED TO COME TOGETHER AND FIGURE OUT THE POWER SUPPLY/CIRCUIT FOR DRIVING THE BOARD AND LEDs"

Commit message: Added unified power, caps, Data in resistor. Modified placements to match enclosure I/O git status
Parts:
- removed TP1, TP2: TestPoint_Alt, TestPoint:TestPoint_Pad_1.5x1.5mm
- added C1: 470u, Capacitor_THT:CP_Radial_D8.0mm_P3.80mm, F.Cu at (54.6, 119.4)
- added C2: 0.1u, Capacitor_THT:C_Disc_D4.7mm_W2.5mm_P5.00mm, F.Cu at (36.8, 80.0)
- added J2: 5V, 4A DC, EQLightBarLibrary:PJ047BH DC Jack, F.Cu at (95.7, 79.8)
- added R1: 330, Resistor_THT:R_Axial_DIN0207_L6.3mm_D2.5mm_P7.62mm_Horizontal, F.Cu at (44.5, 115.6)
- moved U4 30.4 mm to (64.8, 108.1), turned to -90 degrees
- moved U2 23.3 mm to (45.7, 44.5)
- moved U1 21.6 mm to (29.2, 91.4)
- moved REF** 2.11 mm to (177.0, 106.0)
- moved REF** 0.84 mm to (31.0, 73.0)
- moved REF** 0.68 mm to (324.0, 73.0)
- moved REF** 0.67 mm to (31.0, 138.0)
- moved REF** 0.46 mm to (324.0, 138.0)
Connections:
- net 5V USB renamed 5V DC
- U1 pad GND1: Net-(U1-GND) -> GND
- U1 pad GND3: Net-(U1-GND__2) -> GND
- U2 pad G: Net-(U1-GND__2) -> GND
- U2 pad GND: Net-(U1-GND) -> GND
- U4 pad 2: /CLOCK -> /3.3V DATA
- U4 pad 3: Net-(D1-CI) -> Net-(U4-1Y)
- U4 pad 5: /3.3V DATA -> /CLOCK
- U4 pad 6: Net-(D1-DI) -> Net-(D1-CI)
Routing:
- net 5V DC: track 0.00 -> 139.5 mm
- net /CLOCK: track 78.0 -> 7.18 mm
- net /3.3V DATA: track 66.5 -> 5.08 mm
- net Net-(D1-CI): track 12.0 -> 57.7 mm
- net Net-(U4-1Y): track 0.00 -> 27.6 mm
- net Net-(D1-DI): track 14.6 -> 17.7 mm
- net unconnected-(U1-OUT1B-Pad32): track 0.00 -> 0.53 mm
- removed copper zone on B.Cu, net (none)
- removed copper zone on F.Cu, net (none)
Other:
- board size 300 x 71.4 mm -> 299 x 71.4 mm
- board text removed: "WE REALLY REALLY NEED TO COME TOGETHER AND FIGURE OUT THE POWER SUPPLY/CIRCUIT FOR DRIVING THE BOARD AND LEDs"
